File: Initial layout.brd (EAGLE design)
At the start: 153.3 x 128.3 mm, 50 parts, among them U2 TPS54540DDARQ1

Commit message: Worked on connecor pin
Connections:
- new net AMS: U$1.P$20, U$2.5
- new net BSPD: U$1.P$22, U$2.7
- new net IMD: U$1.P$21, U$2.6
- new net N$16: U$2.3V3
- new net N$19: U$2.24
- new net N$20: H1.2
- new net N$21: H1.3
- new net N$22: H1.4
- new net N$23: H1.5
- new net N$24: H1.6
- new net N$27: LED1.4-DIN, U$2.2
- new net SW_BIT0: U$1.P$13, U$2.14/A0
- new net SW_BIT1: U$1.P$14, U$2.15/A1
- new net SW_BIT2: U$1.P$15, U$2.16/A2
- new net SW_BIT3: U$1.P$17, U$2.17/A3
- new net TPS: U$1.P$23, U$2.8
- net +3V3: no longer H1.1, U$2.3V3
- net +5V: now also U$1.P$18
- net CANH1: now also U$1.P$10; no longer U$1.P$9
- net CANL1: now also U$1.P$9; no longer U$1.P$10
- net GND: now also U$1.P$19
- net N$11: now also H1.1; no longer H1.2, U$2.24
- net N$13: no longer H1.3
- net N$15: no longer H1.4
- net N$17: no longer H1.5
- net N$18: no longer H1.6
Changed lines of the file:
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@@
 <contactref element="U3" pad="8"/>
 <contactref element="C20" pad="2"/>
+<contactref element="U$1" pad="P$19"/>
 <wire x1="-135.24" y1="-109.22" x2="-135.24" y2="-114.3" width="0" layer="19" extent="1-1"/>
 <wire x1="-135.24" y1="-104.14" x2="-135.24" y2="-109.22" width="0" layer="19" extent="1-1"/>
@@
 <wire x1="-135.24" y1="-58.42" x2="-135.24" y2="-63.5" width="0" layer="19" extent="1-1"/>
 <wire x1="-130.81" y1="-48.26" x2="-135.24" y2="-58.42" width="0" layer="19" extent="1-1"/>
-<wire x1="-93" y1="-128.96" x2="-135.24" y2="-114.3" width="0" layer="19" extent="1-1"/>
-<wire x1="-85.09" y1="-40.64" x2="-130.81" y2="-48.26" width="0" layer="19" extent="1-1"/>
-<wire x1="-134.25" y1="-163.936" x2="-135.24" y2="-114.3" width="0" layer="19" extent="1-1"/>
+<wire x1="-105" y1="-128.96" x2="-135.24" y2="-114.3" width="0" layer="19" extent="1-1"/>
+<wire x1="-93" y1="-128.96" x2="-105" y2="-128.96" width="0" layer="19" extent="1-1"/>
+<wire x1="-134.25" y1="-163.936" x2="-105" y2="-128.96" width="0" layer="19" extent="1-1"/>
 <wire x1="-130.4" y1="-179.095" x2="-134.25" y2="-163.936" width="0" layer="19" extent="1-1"/>
 <wire x1="-135.6" y1="-180.365" x2="-130.4" y2="-179.095" width="0" layer="19" extent="1-1"/>
 <wire x1="-130.05" y1="-187" x2="-130.4" y2="-179.095" width="0" layer="19" extent="1-1"/>
 <wire x1="-135.05" y1="-194" x2="-130.05" y2="-187" width="0" layer="19" extent="1-1"/>
+<wire x1="-85.09" y1="-40.64" x2="-130.81" y2="-48.26" width="0" layer="19" extent="1-1"/>
 <wire x1="-75.6412" y1="12.2936" x2="-85.09" y2="-40.64" width="0" layer="19" extent="1-1"/>
 <wire x1="-19.3548" y1="67.5132" x2="-19.3548" y2="67.3608" width="0" layer="19" extent="1-1"/>
@@
 <contactref element="C19" pad="1"/>
 <contactref element="U$2" pad="VIN"/>
+<contactref element="U$1" pad="P$18"/>
 <wire x1="-136.54" y1="-109.22" x2="-136.54" y2="-114.3" width="0" layer="19" extent="1-1"/>
 <wire x1="-136.54" y1="-104.14" x2="-136.54" y2="-109.22" width="0" layer="19" extent="1-1"/>
@@
 <wire x1="-136.54" y1="-58.42" x2="-136.54" y2="-63.5" width="0" layer="19" extent="1-1"/>
 <wire x1="-130.81" y1="-33.02" x2="-136.54" y2="-58.42" width="0" layer="19" extent="1-1"/>
-<wire x1="-135.6" y1="-181.635" x2="-136.54" y2="-114.3" width="0" layer="19" extent="1-1"/>
+<wire x1="-101" y1="-128.96" x2="-136.54" y2="-114.3" width="0" layer="19" extent="1-1"/>
+<wire x1="-135.6" y1="-181.635" x2="-101" y2="-128.96" width="0" layer="19" extent="1-1"/>
 <wire x1="-131.95" y1="-187" x2="-135.6" y2="-181.635" width="0" layer="19" extent="1-1"/>
 <wire x1="-74.08" y1="16.51" x2="-130.81" y2="-33.02" width="0" layer="19" extent="1-1"/>
@@
 </signal>
 <signal name="+3V3">
-<contactref element="H1" pad="1"/>
-<contactref element="U$2" pad="3V3"/>
 <contactref element="U3" pad="5"/>
 <contactref element="C20" pad="1"/>
-<wire x1="-123.75" y1="-163.936" x2="-95.25" y2="-48.26" width="0" layer="19" extent="1-1"/>
-<wire x1="-130.4" y1="-182.905" x2="-123.75" y2="-163.936" width="0" layer="19" extent="1-1"/>
-<wire x1="-136.95" y1="-194" x2="-130.4" y2="-182.905" width="0" layer="19" extent="1-1"/>
-</signal>
-<signal name="N$11">
-<contactref element="U$2" pad="24"/>
-<contactref element="H1" pad="2"/>
-<wire x1="-125.25" y1="-163.936" x2="-92.71" y2="-48.26" width="0" layer="19" extent="1-1"/>
+<wire x1="-130.4" y1="-182.905" x2="-136.95" y2="-194" width="0" layer="19" extent="1-1"/>
 </signal>
 <signal name="N$13">
 <contactref element="U$2" pad="25"/>
-<contactref element="H1" pad="3"/>
-<wire x1="-126.75" y1="-163.936" x2="-90.17" y2="-48.26" width="0" layer="19" extent="1-1"/>
 </signal>
 <signal name="N$15">
 <contactref element="U$2" pad="26"/>
-<contactref element="H1" pad="4"/>
-<wire x1="-128.25" y1="-163.936" x2="-87.63" y2="-48.26" width="0" layer="19" extent="1-1"/>
 </signal>
 <signal name="N$17">
 <contactref element="U$2" pad="27"/>
-<contactref element="H1" pad="5"/>
-<wire x1="-129.75" y1="-163.936" x2="-85.09" y2="-48.26" width="0" layer="19" extent="1-1"/>
 </signal>
 <signal name="N$18">
 <contactref element="U$2" pad="28"/>
+</signal>
+<signal name="CANL1">
+<contactref element="U3" pad="6"/>
+<contactref element="R4" pad="2"/>
+<contactref element="U$1" pad="P$9"/>
+<wire x1="-130.4" y1="-181.635" x2="-95" y2="-132.96" width="0" layer="19" extent="1-1"/>
+<wire x1="-135.05" y1="-187" x2="-130.4" y2="-181.635" width="0" layer="19" extent="1-1"/>
+</signal>
+<signal name="N$3">
+<contactref element="U$2" pad="31/A12"/>
+<contactref element="H1" pad="7"/>
+<wire x1="-132.75" y1="-163.936" x2="-74.93" y2="-48.26" width="0" layer="19" extent="1-1"/>
+</signal>
+<signal name="N$16">
+<contactref element="U$2" pad="3V3"/>
+</signal>
+<signal name="N$19">
+<contactref element="U$2" pad="24"/>
+</signal>
+<signal name="N$11">
+<contactref element="H1" pad="1"/>
+</signal>
+<signal name="N$20">
+<contactref element="H1" pad="2"/>
+</signal>
+<signal name="N$21">
+<contactref element="H1" pad="3"/>
+</signal>
+<signal name="N$22">
+<contactref element="H1" pad="4"/>
+</signal>
+<signal name="N$23">
+<contactref element="H1" pad="5"/>
+</signal>
+<signal name="N$24">
 <contactref element="H1" pad="6"/>
-<wire x1="-131.25" y1="-163.936" x2="-82.55" y2="-48.26" width="0" layer="19" extent="1-1"/>
-</signal>
-<signal name="N$25">
+</signal>
+<signal name="CANH1">
+<contactref element="U3" pad="7"/>
+<contactref element="R4" pad="1"/>
+<contactref element="U$1" pad="P$10"/>
+<wire x1="-130.4" y1="-180.365" x2="-99" y2="-132.96" width="0" layer="19" extent="1-1"/>
+<wire x1="-136.95" y1="-187" x2="-130.4" y2="-180.365" width="0" layer="19" extent="1-1"/>
+</signal>
+<signal name="N$28">
+<contactref element="U3" pad="1"/>
+<contactref element="U$2" pad="3/CANTX"/>
+<wire x1="-135.6" y1="-179.095" x2="-120.65" y2="-48.26" width="0" layer="19" extent="1-1"/>
+</signal>
+<signal name="N$26">
 <contactref element="U3" pad="4"/>
 <contactref element="U$2" pad="4/CANRX"/>
 <wire x1="-135.6" y1="-182.905" x2="-118.11" y2="-48.26" width="0" layer="19" extent="1-1"/>
 </signal>
-<signal name="N$26">
-<contactref element="U3" pad="1"/>
-<contactref element="U$2" pad="3/CANTX"/>
-<wire x1="-135.6" y1="-179.095" x2="-120.65" y2="-48.26" width="0" layer="19" extent="1-1"/>
-</signal>
-<signal name="CANL1">
-<contactref element="U3" pad="6"/>
-<contactref element="R4" pad="2"/>
-<contactref element="U$1" pad="P$10"/>
-<wire x1="-130.4" y1="-181.635" x2="-99" y2="-132.96" width="0" layer="19" extent="1-1"/>
-<wire x1="-135.05" y1="-187" x2="-130.4" y2="-181.635" width="0" layer="19" extent="1-1"/>
-</signal>
-<signal name="CANH1">
-<contactref element="U3" pad="7"/>
-<contactref element="R4" pad="1"/>
-<contactref element="U$1" pad="P$9"/>
-<wire x1="-130.4" y1="-180.365" x2="-95" y2="-132.96" width="0" layer="19" extent="1-1"/>
-<wire x1="-136.95" y1="-187" x2="-130.4" y2="-180.365" width="0" layer="19" extent="1-1"/>
-</signal>
-<signal name="N$3">
-<contactref element="H1" pad="7"/>
-<contactref element="U$2" pad="31/A12"/>
-<wire x1="-132.75" y1="-163.936" x2="-74.93" y2="-48.26" width="0" layer="19" extent="1-1"/>
+<signal name="N$27">
+<contactref element="U$2" pad="2"/>
+<contactref element="LED1" pad="4-DIN"/>
+<wire x1="-11.05" y1="67.4" x2="-123.19" y2="-48.26" width="0" layer="19" extent="1-1"/>
+</signal>
+<signal name="SW_BIT3">
+<contactref element="U$1" pad="P$17"/>
+<contactref element="U$2" pad="17/A3"/>
+<wire x1="-107.95" y1="-33.02" x2="-97" y2="-128.96" width="0" layer="19" extent="1-1"/>
+</signal>
+<signal name="AMS">
+<contactref element="U$2" pad="5"/>
+<contactref element="U$1" pad="P$20"/>
+<wire x1="-115.57" y1="-48.26" x2="-109" y2="-128.96" width="0" layer="19" extent="1-1"/>
+</signal>
+<signal name="IMD">
+<contactref element="U$2" pad="6"/>
+<contactref element="U$1" pad="P$21"/>
+<wire x1="-113.03" y1="-48.26" x2="-113" y2="-128.96" width="0" layer="19" extent="1-1"/>
+</signal>
+<signal name="BSPD">
+<contactref element="U$2" pad="7"/>
+<contactref element="U$1" pad="P$22"/>
+<wire x1="-110.49" y1="-48.26" x2="-117" y2="-128.96" width="0" layer="19" extent="1-1"/>
+</signal>
+<signal name="TPS">
+<contactref element="U$2" pad="8"/>
+<contactref element="U$1" pad="P$23"/>
+<wire x1="-107.95" y1="-48.26" x2="-121" y2="-128.96" width="0" layer="19" extent="1-1"/>
+</signal>
+<signal name="SW_BIT2">
+<contactref element="U$1" pad="P$15"/>
+<contactref element="U$2" pad="16/A2"/>
+<wire x1="-105.41" y1="-33.02" x2="-119" y2="-132.96" width="0" layer="19" extent="1-1"/>
+</signal>
+<signal name="SW_BIT1">
+<contactref element="U$1" pad="P$14"/>
+<contactref element="U$2" pad="15/A1"/>
+<wire x1="-102.87" y1="-33.02" x2="-115" y2="-132.96" width="0" layer="19" extent="1-1"/>
+</signal>
+<signal name="SW_BIT0">
+<contactref element="U$1" pad="P$13"/>
+<contactref element="U$2" pad="14/A0"/>
+<wire x1="-100.33" y1="-33.02" x2="-111" y2="-132.96" width="0" layer="19" extent="1-1"/>
 </signal>
 </signals>

Commit message: Finished Schematic?? Probably.
Parts:
- moved U$1 256.3 mm to (94.0, 26.0)
- moved U$2 216.5 mm to (92.1, 53.4)
Connections:
- new net LBL: U$1.P$5, U$2.31/A12
- new net RTDL: U$1.P$4, U$2.30
- new net SERVO_PWM: U$1.P$3, U$2.29
- net +5V: now also U$1.P$2
- net GND: now also U$1.P$6
- net N$3: now also U$2.32/A13; no longer U$2.31/A12

Commit message: Rough board work
Parts:
- moved C19 411.8 mm to (125.3, 135.4)
- moved C20 394.6 mm to (78.2, 137.4)
- moved H1 367.7 mm to (116.8, 105.4)
- moved U3 366.2 mm to (95.2, 105.4)
- moved R4 360.6 mm to (94.4, 90.4)
- moved C1 354.7 mm to (169.2, 122.5)
- moved C7 350.6 mm to (144.5, 121.6)
- moved C6 344.5 mm to (144.3, 116.6)
- moved C5 340.0 mm to (145.2, 112.6)
- moved C16 335.7 mm to (127.0, 94.5)
- moved C15 331.9 mm to (145.1, 67.5)
- moved C14 328.4 mm to (127.2, 92.5)
- moved C13 323.7 mm to (127.2, 89.5)
- moved C11 319.2 mm to (127.3, 86.5)
- moved C3 317.6 mm to (145.6, 78.5)
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Routing:
- net GND: track 424.1 -> 0.00 mm
- net +5V: track 386.3 -> 0.00 mm, vias 3 -> 0
- net X-: track 93.7 -> 0.00 mm
- net Y+: track 80.5 -> 0.00 mm
- net X+: track 78.7 -> 0.00 mm, vias 2 -> 0
- net CS: track 77.3 -> 0.00 mm
- net RST: track 72.8 -> 0.00 mm
- net Y-: track 71.2 -> 0.00 mm
- net SW_5V: track 54.4 -> 0.00 mm, vias 4 -> 0
- net FB_5V: track 39.4 -> 0.00 mm
- net N$39: track 37.5 -> 0.00 mm
- net COMP_5V: track 37.1 -> 0.00 mm, vias 2 -> 0
- net BOOT_5V: track 33.6 -> 0.00 mm, vias 2 -> 0
- net +15V: track 30.6 -> 0.00 mm, vias 2 -> 0
- net 5VREG_EN: track 23.7 -> 0.00 mm, vias 2 -> 0
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Other:
- board size 153.3 x 128.3 mm -> 152.4 x 127 mm

Commit message: Finished Schematic
Connections:
- new net SPARE_1: U$1.P$12, U$2.33/A14
- new net SPARE_2: U$1.P$11, U$2.34/A15
- new net SPARE_3: U$1.P$8, U$2.35/A16
- new net SPARE_4: U$1.P$7, U$2.36/A17
Changed lines of the file:
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@@
 <wire x1="41.85" y1="125.73" x2="123.64" y2="102.09" width="0" layer="19" extent="16-16"/>
+</signal>
+<signal name="SPARE_1">
+<contactref element="U$2" pad="33/A14"/>
+<contactref element="U$1" pad="P$12"/>
+<wire x1="109.22" y1="67.35" x2="72.84" y2="117.33" width="0" layer="19" extent="1-1"/>
+</signal>
+<signal name="SPARE_2">
+<contactref element="U$2" pad="34/A15"/>
+<contactref element="U$1" pad="P$11"/>
+<wire x1="113.22" y1="67.35" x2="75.38" y2="117.33" width="0" layer="19" extent="1-1"/>
+</signal>
+<signal name="SPARE_3">
+<contactref element="U$2" pad="35/A16"/>
+<contactref element="U$1" pad="P$8"/>
+<wire x1="95.22" y1="63.35" x2="77.92" y2="117.33" width="0" layer="19" extent="1-1"/>
+</signal>
+<signal name="SPARE_4">
+<contactref element="U$2" pad="36/A17"/>
+<contactref element="U$1" pad="P$7"/>
+<wire x1="99.22" y1="63.35" x2="80.46" y2="117.33" width="0" layer="19" extent="1-1"/>
 </signal>
 </signals>

Commit message: Begin Board layout
Parts:
- moved R6 167.1 mm to (210.8, 39.4)
- moved U2 156.6 mm to (239.1, 26.4), turned to 90 degrees
- moved D6 155.7 mm to (223.1, 33.4)
- moved C8 145.3 mm to (205.6, 39.4)
- moved C24 143.9 mm to (205.7, 26.4)
- moved C19 131.8 mm to (2.62, 87.3), turned to 90 degrees
- moved L3 128.7 mm to (238.1, 35.0)
- moved C1 126.0 mm to (43.5, 130.8), turned to 270 degrees
- moved C9 123.4 mm to (206.1, 34.4)
- moved U$1 121.1 mm to (230.2, 63.3)
- moved R29 117.2 mm to (223.2, 25.4)
- moved R28 116.5 mm to (219.6, 25.4)
- moved C18 110.4 mm to (211.6, 29.2), turned to 180 degrees
- moved C2 106.3 mm to (54.5, 137.6), turned to 270 degrees
- moved C3 100.6 mm to (65.5, 139.4), turned to 270 degrees
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Routing:
- net N$5: track 0.00 -> 41.6 mm, vias 0 -> 2
- net N$6: track 0.00 -> 40.8 mm
- net N$4: track 0.00 -> 38.2 mm, vias 0 -> 2
- net N$39: track 0.00 -> 36.9 mm, vias 0 -> 2
- net N$8: track 0.00 -> 36.5 mm, vias 0 -> 2
- net N$2: track 0.00 -> 36.1 mm, vias 0 -> 2
- net N$36: track 0.00 -> 35.7 mm, vias 0 -> 2
- net N$38: track 0.00 -> 35.2 mm, vias 0 -> 2
- net N$37: track 0.00 -> 33.8 mm, vias 0 -> 2
- net N$40: track 0.00 -> 33.1 mm
- net +5V: track 0.00 -> 32.1 mm, vias 0 -> 12
- net N$7: track 0.00 -> 31.8 mm, vias 0 -> 2
- net +3V3: track 0.00 -> 4.27 mm
- net CANH1: track 0.00 -> 3.75 mm
- net CANL1: track 0.00 -> 3.57 mm
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