File: Right Ear Board.sch (EAGLE design)
At the start: 6 parts, among them J1 502585-0470

Commit message: Brandon did a thing
Changed lines of the file:
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@@
 <part name="GND1" library="supply1" deviceset="GND" device=""/>
 <part name="J1" library="FormE" deviceset="MOLEX_CLICKMATE-4-R/A" device="" value="502585-0470"/>
+<part name="GND2" library="supply1" deviceset="GND" device=""/>
+<part name="GND3" library="supply1" deviceset="GND" device=""/>
+<part name="GND4" library="supply1" deviceset="GND" device=""/>
+<part name="GND5" library="supply1" deviceset="GND" device=""/>
+<part name="P+1" library="supply1" library_urn="urn:adsk.eagle:library:371" deviceset="+5V" device=""/>
+<part name="P+2" library="supply1" library_urn="urn:adsk.eagle:library:371" deviceset="+5V" device=""/>
+<part name="P+3" library="supply1" library_urn="urn:adsk.eagle:library:371" deviceset="+5V" device=""/>
 </parts>
 <sheets>
@@
 <instance part="GND1" gate="1" x="128.27" y="87.63"/>
 <instance part="J1" gate="G$1" x="165.1" y="49.53"/>
+<instance part="GND2" gate="1" x="58.42" y="61.976"/>
+<instance part="GND3" gate="1" x="106.68" y="61.214"/>
+<instance part="GND4" gate="1" x="91.186" y="34.29"/>
+<instance part="GND5" gate="1" x="151.13" y="41.91"/>
+<instance part="P+1" gate="1" x="152.4" y="60.96"/>
+<instance part="P+2" gate="1" x="53.34" y="106.68"/>
+<instance part="P+3" gate="1" x="86.36" y="58.42"/>
 </instances>
 <busses>
@@
 <wire x1="86.36" y1="49.53" x2="86.36" y2="55.88" width="0.1524" layer="91"/>
 <label x="87.63" y="55.88" size="1.778" layer="95"/>
+<pinref part="P+3" gate="1" pin="+5V"/>
 </segment>
 <segment>
@@
 <pinref part="LED7" gate="G$1" pin="VDD"/>
 <wire x1="53.34" y1="97.79" x2="53.34" y2="100.33" width="0.1524" layer="91"/>
-<label x="54.61" y="104.14" size="1.778" layer="95"/>
 <wire x1="53.34" y1="100.33" x2="53.34" y2="104.14" width="0.1524" layer="91"/>
 <wire x1="81.28" y1="100.33" x2="53.34" y2="100.33" width="0.1524" layer="91"/>
@@
 <wire x1="101.6" y1="100.33" x2="128.27" y2="100.33" width="0.1524" layer="91"/>
 <wire x1="128.27" y1="100.33" x2="128.27" y2="97.79" width="0.1524" layer="91"/>
+<pinref part="P+2" gate="1" pin="+5V"/>
 </segment>
 <segment>
@@
 <wire x1="162.56" y1="54.61" x2="152.4" y2="54.61" width="0.1524" layer="91"/>
 <wire x1="152.4" y1="54.61" x2="152.4" y2="58.42" width="0.1524" layer="91"/>
-<label x="152.4" y="58.42" size="1.778" layer="95"/>
+<pinref part="P+1" gate="1" pin="+5V"/>
 </segment>
 </net>
 <net name="GND" class="0">
-<segment>
-<pinref part="LED7" gate="G$1" pin="GND"/>
-<wire x1="58.42" y1="72.39" x2="58.42" y2="66.04" width="0.1524" layer="91"/>
-<label x="60.96" y="66.04" size="1.778" layer="95"/>
-</segment>
-<segment>
-<pinref part="SV1" gate="G$1" pin="3"/>
-<wire x1="86.36" y1="44.45" x2="86.36" y2="38.1" width="0.1524" layer="91"/>
-<label x="87.63" y="38.1" size="1.778" layer="95"/>
-</segment>
-<segment>
-<pinref part="LED1" gate="G$1" pin="GND"/>
-<wire x1="106.68" y1="72.39" x2="106.68" y2="66.04" width="0.1524" layer="91"/>
-<label x="109.22" y="66.04" size="1.778" layer="95"/>
-</segment>
 <segment>
 <pinref part="C1" gate="G$1" pin="2"/>
@@
 <segment>
 <pinref part="J1" gate="G$1" pin="4"/>
-<wire x1="162.56" y1="46.99" x2="152.4" y2="46.99" width="0.1524" layer="91"/>
-<wire x1="152.4" y1="46.99" x2="152.4" y2="44.45" width="0.1524" layer="91"/>
-<label x="152.4" y="44.45" size="1.778" layer="95"/>
+<wire x1="162.56" y1="46.99" x2="151.13" y2="46.99" width="0.1524" layer="91"/>
+<pinref part="GND5" gate="1" pin="GND"/>
+<wire x1="151.13" y1="46.99" x2="151.13" y2="44.45" width="0.1524" layer="91"/>
+</segment>
+<segment>
+<pinref part="LED7" gate="G$1" pin="GND"/>
+<pinref part="GND2" gate="1" pin="GND"/>
+<wire x1="58.42" y1="72.39" x2="58.42" y2="64.516" width="0.1524" layer="91"/>
+</segment>
+<segment>
+<pinref part="LED1" gate="G$1" pin="GND"/>
+<pinref part="GND3" gate="1" pin="GND"/>
+<wire x1="106.68" y1="72.39" x2="106.68" y2="63.754" width="0.1524" layer="91"/>
+</segment>
+<segment>
+<pinref part="SV1" gate="G$1" pin="3"/>
+<pinref part="GND4" gate="1" pin="GND"/>
+<wire x1="86.36" y1="44.45" x2="91.186" y2="44.45" width="0.1524" layer="91"/>
+<wire x1="91.186" y1="44.45" x2="91.186" y2="36.83" width="0.1524" layer="91"/>
 </segment>
 </net>
