File: Center Dash/RJ-45 Dash Daughter Board.brd (EAGLE design)
At the start: 35.5 x 36.5 mm, 3 parts, among them J1 5025840470

Commit message: Done with board layouts
Parts:
- moved U$1 12.0 mm to (71.1, 86.4), turned to 180 degrees
Routing:
- net N$9: track 18.8 -> 58.9 mm, vias 0 -> 2
- net N$7: track 45.7 -> 20.6 mm, vias 0 -> 1
- net N$4: track 35.2 -> 17.0 mm, vias 0 -> 1
- net N$8: track 35.7 -> 18.9 mm, vias 0 -> 1
- net N$12: track 32.8 -> 18.0 mm
- net N$6: track 30.4 -> 17.2 mm, vias 0 -> 1
- net N$10: track 19.3 -> 29.9 mm, vias 0 -> 1
- net N$3: track 27.7 -> 18.0 mm
- net N$11: track 30.7 -> 21.2 mm, vias 0 -> 1
- net N$2: track 24.7 -> 16.1 mm
- net N$1: track 21.7 -> 17.8 mm
- net N$5: track 23.0 -> 20.4 mm
