File: Center Dash/Center Dash.sch (EAGLE design)
At the start: 90 parts, among them J1 502585-0470, Q1 BSS138, Q2 BSS138, Q3 BSS138, Q4 BSS138, U1 ADG3304BRUZ-REEL7, U2 TPS54540DDARQ1

Commit message: last minute fix again
Connections:
- net +3V3: now also U1.EN
Changed lines of the file:
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@@
 </part>
 <part name="GND37" library="supply1" deviceset="GND" device=""/>
+<part name="+3V6" library="supply1" library_urn="urn:adsk.eagle:library:371" deviceset="+3V3" device=""/>
 </parts>
 <sheets>
@@
 </instance>
 <instance part="GND37" gate="1" x="340.36" y="-271.78"/>
+<instance part="+3V6" gate="G$1" x="203.2" y="-175.26"/>
 </instances>
 <busses>
@@
 <pinref part="+3V5" gate="G$1" pin="+3V3"/>
 </segment>
-</net>
+<segment>
+<pinref part="U1" gate="G$1" pin="EN"/>
+<wire x1="208.28" y1="-180.34" x2="203.2" y2="-180.34" width="0.1524" layer="91"/>
+<wire x1="203.2" y1="-180.34" x2="203.2" y2="-177.8" width="0.1524" layer="91"/>
+<pinref part="+3V6" gate="G$1" pin="+3V3"/>
+</segment>
+</net>
